Commit message: finish API

File: urdf/ur5_robot.urdf (robot description, URDF)
Before this commit: robot ur5, 9 links, 8 joints
Links:
- added link base
- added link tool0
Joints:
- added joint base_link-base_fixed_joint: type fixed, parent base_link, child base, origin xyz=0 0 0 rpy=0 0 -3.14159265
- added joint wrist_3_link-tool0_fixed_joint: type fixed, parent wrist_3_link, child tool0, origin xyz=0 0.0823 0 rpy=-1.570796325 0 0
- joint elbow_joint: limit lower=-3.14159265 upper=3.14159265 effort=150.0 velocity=3.15 -> lower=-6.2831853 upper=6.2831853 effort=150.0 velocity=3.15
- joint shoulder_lift_joint: limit lower=-3.14159265 upper=3.14159265 effort=150.0 velocity=3.15 -> lower=-6.2831853 upper=6.2831853 effort=150.0 velocity=3.15; origin xyz=0.0 0.13585 0.0 rpy=0.0 1.570796325 0.0 -> xyz=0.0 0.13585 0.0 rpy=0.0 0.0 0.0
- joint shoulder_pan_joint: limit lower=-3.14159265 upper=3.14159265 effort=150.0 velocity=3.15 -> lower=-6.2831853 upper=6.2831853 effort=150.0 velocity=3.15
- joint wrist_1_joint: limit lower=-3.14159265 upper=3.14159265 effort=28.0 velocity=3.2 -> lower=-6.2831853 upper=6.2831853 effort=28.0 velocity=3.2; origin xyz=0.0 0.0 0.39225 rpy=0.0 1.570796325 0.0 -> xyz=0.0 0.0 0.39225 rpy=0.0 0.0 0.0
- joint wrist_2_joint: limit lower=-3.14159265 upper=3.14159265 effort=28.0 velocity=3.2 -> lower=-6.2831853 upper=6.2831853 effort=28.0 velocity=3.2
- joint wrist_3_joint: limit lower=-3.14159265 upper=3.14159265 effort=28.0 velocity=3.2 -> lower=-6.2831853 upper=6.2831853 effort=28.0 velocity=3.2
